Commit message: fix head settle time, dataframe index check, rh8d translation

File: urdf/rh8d.urdf (robot description, URDF)
Before this commit: robot rh8d, 27 links, 26 joints
Joints:
- joint joint_base: origin xyz=0 0 0 rpy=0 0 0 -> xyz=0 0 0.007 rpy=0 0 0

Commit message: fix rh8d tf

File: urdf/rh8d.urdf (robot description, URDF)
Before this commit: robot rh8d, 27 links, 26 joints
Joints:
- joint jointI1: origin xyz=-0.0043044918 0.0812907302 0.0367863551 rpy=-0.08267713  0.17715231 -2.93857995 -> xyz=-0.0043044918 0.0812907302 0.0367863551 rpy=-0.1 0.17715231 -2.85
- joint jointI2: origin xyz=0 -0.0258749732 0 rpy=0 0 -0.015 -> xyz=0 -0.0258749732 0 rpy=0 0 0.15
- joint jointI3: origin xyz=0 -0.0258749732 0 rpy=0 0 0 -> xyz=0 -0.0258749732 0 rpy=0 0 0.05
- joint jointL1: origin xyz=-0.0031705239 0.0731417977 -0.0376310382 rpy=0.14 -0.17  -2.95156384 -> xyz=-0.0031705239 0.0731417977 -0.0376310382 rpy=0.2 -0.17  -2.9
- joint jointL2: origin xyz=0 -0.0258749732 0 rpy=0 0 -0.015 -> xyz=0 -0.0258749732 0 rpy=0 0 0.1
- joint jointL3: origin xyz=0 -0.0258749732 0 rpy=0 0 0 -> xyz=0 -0.0258749732 0 rpy=0 0 0.0
- joint jointM1: origin xyz=-0.0012008743 0.0828960623 0.0118294206 rpy=-0.02 0.06 -2.92246721 -> xyz=-0.0012008743 0.0828960623 0.0118294206 rpy=0.0 0.06 -2.85
- joint jointM2: origin xyz=0 -0.0258749732 0 rpy=0 0 -0.015 -> xyz=0 -0.0258749732 0 rpy=0 0 0.15
- joint jointM3: origin xyz=0 -0.0258749732 0 rpy=0 0 0 -> xyz=0 -0.0258749732 0 rpy=0 0 0.05
- joint jointR1: origin xyz=-0.0011171786 0.0818708881 -0.0130285291 rpy=0.06 -0.04 -2.92922802 -> xyz=-0.0011171786 0.0818708881 -0.0130285291 rpy=0.0 -0.04 -2.9
- joint jointR2: origin xyz=0 -0.0258749732 0 rpy=0 0 -0.015 -> xyz=0 -0.0258749732 0 rpy=0 0 0.0
- joint jointR3: origin xyz=0 -0.0258749732 0 rpy=0 0 0 -> xyz=0 -0.0258749732 0 rpy=0 0 0.0
- joint jointT0: origin xyz=-0.0083412575 0.0157859987 0.0379541955 rpy=-2.54680616 -0.60124514  0.33418237 -> xyz=-0.0083412575 0.0157859987 0.0379541955 rpy=-2.54680616 -0.60124514 0.33
